File: DI.DO_Shield_for_Arduino/DI.DO_Shield_for_Arduino.sch (KiCad schematic (older format))
At the start: 42 parts, among them J1 CONN_08X2, J10 CONN_08X2, J2 CONN_08X2, J3 CONN_08X2, J4 CONN_08X2, J5 CONN_08X2, J6 CONN_08X2, J7 CONN_08X2, J8 CONN_08X2, J9 CONN_08X2, U1 MCP23S08, U1_A0 JUMPER-SMT_2_NC, U1_A1 JUMPER-SMT_2_NO, U1_A2 JUMPER-SMT_2_NO, U2 MCP23S08, U2_A0 JUMPER-SMT_2_NO, U2_A1 JUMPER-SMT_2_NC, U2_A2 JUMPER-SMT_2_NO

Commit message: add buttons and pots sub-boards, push changes
Parts:
- removed C2: 0.1uF, Capacitors_SMD:C_0805_HandSoldering, symbol C
- removed D1, D2, D3, D4, D5, D6, D7, D8: 1N4148W-TP, digikey-footprints:SOD-123, symbol 1N4148W-TP
- removed J1, J2, J3, J4, J5, J6, J7, J8: CONN_08X2, MyFootprintLib:2X8_SHROUDED_PTH, symbol CONN_08X2
- removed J10, J9: CONN_08X2, SparkFun Connectors:2X8, symbol CONN_08X2
- removed R1, R2: 4.7k, Resistors_SMD:R_0805_HandSoldering, symbol R
- removed RN1: 4609X-101-103LF, digikey-footprints:SIP-9_P2.54mm, symbol 4609X-101-103LF
- removed U1, U2: MCP23S08, Housings_DIP:DIP-18_W7.62mm_Socket, symbol MCP23S08
- removed U1_A0: JUMPER-SMT_2_NC, SparkFun Jumpers:SMT-JUMPER_2_NC_TRACE_SILK, symbol JUMPER-SMT_2_NC
- removed U1_A1, U1_A2: JUMPER-SMT_2_NO, SparkFun Jumpers:SMT-JUMPER_2_NO_SILK, symbol JUMPER-SMT_2_NO
- added INTB1: JUMPER-SMT_3_1-NC, SparkFun Jumpers:SMT-JUMPER_3_1-NC_TRACE_SILK, symbol JUMPER-SMT_3_1-NC
- added J1, J2, J3, J4, J5, J6, J7, J8: Conn_02x05_Odd_Even, SparkFun Connectors:2X5-SHROUDED, symbol Conn_02x05_Odd_Even
- added R11, R12, R13, R14, R7: 2k2, Resistors_SMD:R_0805_HandSoldering, symbol R
- added R3: 10k, Resistors_SMD:R_0805_HandSoldering, symbol R
- added SW1: SW_DIP_x08, Buttons_Switches_SMD:SW_DIP_x8_W6.15mm_Slide_Omron_A6H, symbol SW_DIP_x08
- added U1: MCP23S17, Housings_DIP:DIP-28_W7.62mm_LongPads, symbol MCP23S17
- B1: footprint SparkFun Boards:UNO_R3_SHIELD_ICSP -> MyFootprintLib:ARDUINO_R3
- R10, R8, R9: value 10k -> 2k2
- renumbered INT1 to INTA1, R3 to R1, R4 to R2, R5 to R4, R6 to R5, R7 to R6, U2_A0 to U2_A1, U2_A1 to U2_A2, U2_A2 to U2_A3
Connections:
- net GND: now also U1.10 (GND); no longer R10.2, R8.2, R9.2
- net VCC: now also R10.1, R8.1, R9.1, R11.1, R12.1, R13.1, R14.1, R3.1, R7.1, U1.9 (VCC)
- net at R5.1, U2_A2.2: now also U1.16 (A1)
- net at R4.1, U2_A1.2: now also U1.15 (A0)
- net SCL: now reaches B1.SCL, R2.1
- net SCL: now also SW1.13
- net SDA: now reaches B1.SDA, R1.1
- net SDA: now also SW1.11
- net INT_A: now reaches INTA1.2
- net INT_A: now also SW1.15
- net MOSI: now reaches B1.MOSI
- net MOSI: now also SW1.10
- net MISO: now reaches B1.MISO
- net MISO: now also SW1.9
- net CS: now reaches CS1.2
- net CS: now also SW1.14
- net SCK: now reaches B1.SCK
- net SCK: now also SW1.12
- net at R6.1, U2_A3.2: now also U1.17 (A2)
- net at B1.D3 (*D3), INTA1.1: now also INTB1.3
- net at B1.D2, INTA1.3: now also INTB1.1
- new net: J1.1 (Pin_1), J1.2 (Pin_2), U1.1 (GPB0)
- new net: SW1.3, U1.11 (~CS)
- new net: SW1.4, SW1.5, U1.12 (SCK)
- new net: SW1.6, SW1.7, U1.13 (SI)
- new net: SW1.8, U1.14 (SO)
- new net: R3.2, U1.18 (~RESET)
- new net: SW1.1, U1.19 (INTB)
- new net: J2.1 (Pin_1), J2.2 (Pin_2), U1.2 (GPB1)
- new net: SW1.2, U1.20 (INTA)
- new net: J1.3 (Pin_3), J2.3 (Pin_3), J3.3 (Pin_3), J4.3 (Pin_3), J5.3 (Pin_3), J6.3 (Pin_3), J7.3 (Pin_3), J8.3 (Pin_3), R7.2, U1.21 (GPA0)
- new net: J1.5 (Pin_5), J2.5 (Pin_5), J3.5 (Pin_5), J4.5 (Pin_5), J5.5 (Pin_5), J6.5 (Pin_5), J7.5 (Pin_5), J8.5 (Pin_5), R9.2, U1.22 (GPA1)
- new net: J1.7 (Pin_7), J2.7 (Pin_7), J3.7 (Pin_7), J4.7 (Pin_7), J5.7 (Pin_7), J6.7 (Pin_7), J7.7 (Pin_7), J8.7 (Pin_7), R11.2, U1.23 (GPA2)
- new net: J1.9 (Pin_9), J2.9 (Pin_9), J3.9 (Pin_9), J4.9 (Pin_9), J5.10 (Pin_10), J5.9 (Pin_9), J6.10 (Pin_10), J6.9 (Pin_9), J7.10 (Pin_10), J7.9 (Pin_9), J8.4 (Pin_4), J8.9 (Pin_9), R13.2, U1.24 (GPA3)
- new net: J1.4 (Pin_4), J2.4 (Pin_4), J3.4 (Pin_4), J4.4 (Pin_4), R14.2, U1.25 (GPA4)
- new net: J1.6 (Pin_6), J2.6 (Pin_6), J3.6 (Pin_6), J4.6 (Pin_6), J5.8 (Pin_8), J6.8 (Pin_8), J7.8 (Pin_8), J8.6 (Pin_6), R12.2, U1.26 (GPA5)
- new net: J1.8 (Pin_8), J2.8 (Pin_8), J3.8 (Pin_8), J4.8 (Pin_8), J5.6 (Pin_6), J6.6 (Pin_6), J7.6 (Pin_6), J8.8 (Pin_8), R10.2, U1.27 (GPA6)
- new net: J1.10 (Pin_10), J2.10 (Pin_10), J3.10 (Pin_10), J4.10 (Pin_10), J5.4 (Pin_4), J6.4 (Pin_4), J7.4 (Pin_4), J8.10 (Pin_10), R8.2, U1.28 (GPA7)
- new net: J3.1 (Pin_1), J3.2 (Pin_2), U1.3 (GPB2)
- new net: J4.1 (Pin_1), J4.2 (Pin_2), U1.4 (GPB3)
- new net: J5.1 (Pin_1), J5.2 (Pin_2), U1.5 (GPB4)
- new net: J6.1 (Pin_1), J6.2 (Pin_2), U1.6 (GPB5)
- new net: J7.1 (Pin_1), J7.2 (Pin_2), U1.7 (GPB6)
- new net: J8.1 (Pin_1), J8.2 (Pin_2), U1.8 (GPB7)
- new net INT_B: INTB1.2, SW1.16
- no-connect marks 24 -> 22
Other:
- moved on the sheet: B1, C1, CS1, INTA1, R1, R2, R4, R5, R6, U2_A1, U2_A2, U2_A3
