File: MIDI_Shield_16u2/MIDI_shield_16u2.kicad_pcb (KiCad board)
At the start: 2 copper layers, 53.2 x 78.2 mm, 39 parts, among them J1 MIDI_IN, J2 MIDI_OUT, J3 CONN_02, J4 BUZZER_ROUTING_JP, SW1 SW_DIP_x02, U1 OPTO_DARL_6N138S, U2 MCP23S08

Commit message: add buttons and pots sub-boards, push changes
Parts:
- removed D2: 1N4148, Diodes_SMD:D_SOD-123
- removed J3: CONN_02, SparkFun Connectors:1X02
- removed J4: BUZZER_ROUTING_JP, SparkFun Connectors:1X03
- removed KiCad1: KiCad-Logo2_6mm_SilkScreen, Symbols:KiCad-Logo2_6mm_SilkScreen
- removed OSHW1: OSHW-Symbol_13.4x12mm_SilkScreen, Symbols:OSHW-Symbol_13.4x12mm_SilkScreen
- removed h1, h2, h3: >VALUE, MyFootprintLib:Arduino_3.2_connector
- added Q1: Q_NPN_BEC_2222A, TO_SOT_Packages_SMD:SOT-23_Handsoldering, F.Cu at (168.4, 54.6)
- added R11: 10k_1_4W_5%, Resistors_SMD:R_0805_HandSoldering, F.Cu at (176.5, 69.8)
- added REF***: OSHW-Logo2_7.3x6mm_SilkScreen, Symbols:OSHW-Logo2_7.3x6mm_SilkScreen, B.Cu at (161.6, 87.6)
- added REF***: KiCad-Logo2_8mm_SilkScreen, Symbols:KiCad-Logo2_8mm_SilkScreen, B.Cu at (180.9, 84.5)
- B2: footprint MyFootprintLib:UNO_R3_SHIELD_ICSP_16u2_BREAKOUT -> MyFootprintLib:UNO_R3_SHIELD_16u2_BREAKOUT_wHoles
- EXP1, EXP2: footprint SparkFun Connectors:2X5-SHROUDED -> MyFootprintLib:2X5-SHROUDED
- J1, J2: footprint SparkFun Connectors:DIN5-RA-PTH -> MyFootprintLib:DIN5-RA-PTH
- JP1: value MIDI_ROUTING_05X2_JUMPER -> INT; footprint SparkFun Connectors:2X5 -> SparkFun Jumpers:SMT-JUMPER_3_NO_SILK; moved to B.Cu
- JP5: value CONN_06X2PTH -> BUZZER; footprint SparkFun Connectors:2X6 -> SparkFun Jumpers:SMT-JUMPER_3_1-NC_TRACE_SILK; moved to B.Cu
- S1: footprint MyFootprintLib:Switch_Slide_Right_Angle_8.6X4.4mm_EG9559 -> MyFootprintLib:Switch_Slide_Right_Angle_8.6X4.4mm_C&K_OS102011MA1QS1
- SW1: value SW_DIP_x02 -> SW_DIP_x08; footprint Buttons_Switches_THT:SW_DIP_x2_W7.62mm_Slide -> Buttons_Switches_SMD:SW_DIP_x8_W6.15mm_Slide_Omron_A6H
- U1: footprint Housings_DIP:DIP-8_W7.62mm_SMDSocket_SmallPads -> Housings_DIP:DIP-8_W8.89mm_SMDSocket_LongPads
- U2: footprint digikey-footprints:DIP-18_W7.62mm -> Housings_DIP:DIP-18_W7.62mm_Socket_LongPads
- moved JP3 36.5 mm to (160.7, 44.6)
- moved JP2 33.9 mm to (164.5, 44.6)
- moved SW1 27.4 mm to (164.6, 71.2), turned to 180 degrees
- moved JP1 24.9 mm to (154.4, 56.9), turned to 90 degrees
- moved C1 22.1 mm to (186.2, 54.6), turned to 180 degrees
- moved EXP1 21.6 mm to (186.1, 40.6)
- moved EXP2 21.6 mm to (164.5, 40.6)
- moved R2 20.1 mm to (172.2, 83.6), turned to 180 degrees
- moved U2 18.4 mm to (182.1, 57.1), turned to 0 degrees
- moved R8 18.3 mm to (176.5, 72.8)
- moved R6 17.6 mm to (176.5, 67.3), turned to 180 degrees
- moved JP4 13.5 mm to (154.2, 69.3), turned to 270 degrees
- moved D1 11.0 mm to (194.5, 87.2), turned to 90 degrees
- moved R5 10.8 mm to (176.5, 64.8), turned to 180 degrees
- moved JP7 9.81 mm to (156.7, 69.3)
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Connections:
- B2 pad 5V_2: (no net) -> VCC
- B2 pad D2: (no net) -> /EXT_INT0
- B2 pad D9: /EXPANDER_CS -> /LCD&BUZZER_CS
- B2 pad PB4: /16U2_RX -> (no net)
- B2 pad PB5: /16U2_TX -> (no net)
- B2 pad PB6: /16U2_PB6 -> (no net)
- B2 pad PB7: /16U2_PB7 -> (no net)
- B2 pad RX: /328P_RX -> /MIDI_IN
- B2 pad SCK2: /SOFT_SERIAL -> (no net)
- B2 pad TX: /16U2_TX -> /MIDI_OUT
- EXP2 pad 10: (no net) -> /GND_CTL
- JP1 pad 1: /MIDI_IN -> /EXT_INT1
- JP1 pad 2: /16U2_RX -> Net-(JP1-Pad2)
- JP1 pad 3: /MIDI_IN -> /EXT_INT0
- JP5 pad 1: Net-(JP5-Pad1) -> /BUZZER_
- JP5 pad 2: /SDA -> /BUZZER
- JP5 pad 3: Net-(JP5-Pad1) -> /EXT_INT1
- JP9 pad 2: Net-(JP5-Pad10) -> Net-(JP9-Pad2)
- R7 pad 1: Net-(JP5-Pad10) -> Net-(JP9-Pad2)
- R8 pad 1: /LCD_GND_CTL -> Net-(Q1-Pad1)
- R8 pad 2: GND -> /GND_CTL
- S1 pad 1: (no net) -> /16U2_RSTJP
- S1 pad 3: /16U2_RSTJP -> (no net)
- SW1 pad 1: /FAST_SERIAL -> GND
- SW1 pad 2: /SOFT_SERIAL -> /EXPANDER_CS
- SW1 pad 3: GND -> Net-(SW1-Pad3)
- SW1 pad 4: GND -> Net-(SW1-Pad3)
- U2 pad 1: Net-(JP5-Pad5) -> Net-(SW1-Pad3)
- U2 pad 2: Net-(JP5-Pad1) -> Net-(SW1-Pad5)
- U2 pad 3: Net-(JP5-Pad11) -> Net-(SW1-Pad7)
- U2 pad 6: (no net) -> Net-(R11-Pad2)
- U2 pad 8: (no net) -> Net-(JP1-Pad2)
Routing:
- net GND: track 338.6 -> 88.0 mm, vias 21 -> 6
- net /SOFT_SERIAL: track 66.8 -> 0.00 mm
- net /ENC_A_NO: track 90.7 -> 27.4 mm, vias 0 -> 1
- net /ENC_B_NO: track 79.9 -> 26.8 mm, vias 0 -> 1
- net /GND_CTL: track 4.07 -> 55.8 mm, vias 0 -> 1
- net /ENC_BTN: track 19.4 -> 68.0 mm
- net /16U2_TX: track 47.4 -> 0.00 mm
- net /FAST_SERIAL: track 71.3 -> 24.0 mm, vias 0 -> 1
- net /328P_RX: track 46.6 -> 0.00 mm
- net /ENC_B_NC: track 2.55 -> 46.3 mm, vias 0 -> 1
- net Net-(JP1-Pad2): track 0.00 -> 40.2 mm, vias 0 -> 1
- net /SDA: track 71.6 -> 32.0 mm
- net /ENC_A_NC: track 2.49 -> 41.6 mm, vias 0 -> 1
- net /BUZZER: track 9.58 -> 47.1 mm
- net /MIDI_OUT: track 17.4 -> 53.4 mm, vias 0 -> 2
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Other:
- net class Default: via_dia 0.762 -> 0.7; via_drill 0.4064 -> 0.35
- net class PWR: via_dia 0.95 -> 0.85
- board text added: "FST_SER SPI_CS I2C_SCL SPI_SCK I2C_SDA SPI_SI I2C_A2 SPI_SO"
- board text added: "UriShX MIDI.UI Shield v.0.3"
- board text removed: "16U2_PB7 16U2_PB6"
- board text removed: "FAST.SRL SOFT.SRL"
- board text removed: "I2C_SDA SPI_SI I2C_SCL SPI_SCK I2C_A2 SPI_SI"
- board text removed: "MIDI_IN |16U2_SFT.SRL.RX |328P_RX |THRU MIDI_OUT|16U2_SFT.SRL.TX |328P_TX"
