File: MIDI_Shield_16u2/MIDI_shield_16u2.sch (KiCad schematic (older format))
At the start: 34 parts, among them J1 MIDI_IN, J2 MIDI_OUT, J3 CONN_02, J4 BUZZER_ROUTING_JP, SW1 SW_DIP_x02, U1 OPTO_DARL_6N138S, U2 MCP23S08

Commit message: add buttons and pots sub-boards, push changes
Parts:
- removed D2: 1N4148, Diodes_SMD:D_SOD-123, symbol D
- removed J3: CONN_02, SparkFun Connectors:1X02, symbol CONN_02
- removed J4: BUZZER_ROUTING_JP, SparkFun Connectors:1X03, symbol CONN_03
- removed JP1: MIDI_ROUTING_05X2_JUMPER, SparkFun Connectors:2X5, symbol CONN_05X2PTH
- removed JP5: CONN_06X2PTH, SparkFun Connectors:2X6, symbol CONN_06X2SMD_FEMALE
- removed SW1: SW_DIP_x02, Buttons_Switches_THT:SW_DIP_x2_W7.62mm_Slide, symbol SW_DIP_x02
- added JP1: INT, SparkFun Jumpers:SMT-JUMPER_3_NO_SILK, symbol JUMPER-SMT_3_NO
- added JP5: BUZZER, SparkFun Jumpers:SMT-JUMPER_3_1-NC_TRACE_SILK, symbol JUMPER-SMT_3_1-NC
- added Q1: Q_NPN_BEC_2222A, TO_SOT_Packages_SMD:SOT-23_Handsoldering, symbol Q_NPN_BEC
- added R11: 10k_1_4W_5%, Resistors_SMD:R_0805_HandSoldering, symbol RESISTOR0805
- added SW1: SW_DIP_x08, Buttons_Switches_SMD:SW_DIP_x8_W6.15mm_Slide_Omron_A6H, symbol SW_DIP_x08
- B2: footprint MyFootprintLib:UNO_R3_SHIELD_ICSP_16u2_BREAKOUT -> MyFootprintLib:UNO_R3_SHIELD_16u2_BREAKOUT_wHoles
- EXP1, EXP2: footprint SparkFun Connectors:2X5-SHROUDED -> MyFootprintLib:2X5-SHROUDED
- J1, J2: footprint SparkFun Connectors:DIN5-RA-PTH -> MyFootprintLib:DIN5-RA-PTH; Field4 CONN-09481 -> (none)
- S1: footprint MyFootprintLib:Switch_Slide_Right_Angle_8.6X4.4mm_EG9559 -> MyFootprintLib:Switch_Slide_Right_Angle_8.6X4.4mm_C&K_OS102011MA1QS1; Field4 SWCH-10651 -> (none)
- U1: footprint Housings_DIP:DIP-8_W7.62mm_SMDSocket_SmallPads -> Housings_DIP:DIP-8_W8.89mm_SMDSocket_LongPads
- U2: footprint digikey-footprints:DIP-18_W7.62mm -> Housings_DIP:DIP-18_W7.62mm_Socket_LongPads
Connections:
- net 328P_RX is gone; now on net MIDI_IN: B2.RX (D0)
- net 16U2_RSTJP: now also S1.1 (O); no longer S1.3 (S)
- net 16U2_TX: no longer B2.TX (D1)
- net ARDUINO_RST: now also B2.RST (~RESET~)
- net BUZZER: now also JP5.2
- net BUZZER_: now also JP5.1
- net EXPANDER_CS: now also SW1.2; no longer B2.D9 (*D9)
- net EXT_INT0: now also JP1.3
- net EXT_INT1: now also JP1.1, JP5.3
- net FAST_SERIAL: now also SW1.16
- net GND: now also Q1.2 (E), SW1.1; no longer R8.2
- net GND_CTL: now also EXP2.10, R8.2
- net LCD_GND_CTL: now also Q1.3 (C); no longer R8.1
- net MIDI_OUT: now also B2.TX (D1)
- net MISO_: now also SW1.9
- net MOSI_: now also SW1.11
- net SCK_: now also SW1.13
- net SCL: now also SW1.14
- net SDA: now also SW1.12
- net VCC: now also B2.5V_2 (16u2_VCC), R11.1
- net at U2.1 (SCK): now also SW1.3, SW1.4
- net at U2.2 (SI): now also SW1.5, SW1.6
- net at U2.3 (SO): now also SW1.7, SW1.8
- net at U2.6 (~RESET): now also R11.2
- net at U2.8 (INT): now also JP1.2
- net at JP9.2, R7.1: now also SW1.10
- net 16U2_PB6: no longer names the net of B2.PB6
- net 16U2_PB7: no longer names the net of B2.PB7
- net SOFT_SERIAL: no longer names the net of B2.SCK2 (16u2_SCK)
- new net: Q1.1 (B), R8.1
- new net LCD&BUZZER_CS: B2.D9 (*D9), SW1.15
- no-connect marks 25 -> 22
Other:
- moved on the sheet: JP3, R8
