File: MUX_Shield_for_arduino/MUX_Shield_for_arduino.sch (KiCad schematic (older format))
At the start: 30 parts, among them J1 CONN_05X20.05_IN_PTH_SILK, J2 CONN_05X20.05_IN_PTH_SILK, J3 CONN_05X20.05_IN_PTH_SILK, J4 CONN_05X20.05_IN_PTH_SILK, J5 CONN_05X20.05_IN_PTH_SILK, J6 CONN_05X20.05_IN_PTH_SILK, J7 CONN_05X20.05_IN_PTH_SILK, J8 CONN_05X20.05_IN_PTH_SILK, J9 CONN_06X2PTH_FEMALE, U1 74HC4067SM96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

Commit message: add buttons and pots sub-boards, push changes
Parts:
- removed J9: CONN_06X2PTH_FEMALE, SparkFun Connectors:2X6, symbol CONN_06X2PTH_FEMALE
- added JP6: INT, SparkFun Jumpers:SMT-JUMPER_3_NO_SILK, symbol JUMPER-SMT_3_NO
- added R6: 10K, Resistors_SMD:R_0805_HandSoldering, symbol R
- added SW1: SW_DIP_x08, Buttons_Switches_SMD:SW_DIP_x8_W6.15mm_Slide_Omron_A6H, symbol SW_DIP_x08
- J1, J2, J3, J4, J5, J6, J7, J8: footprint SparkFun Connectors:2X5-SHROUDED -> MyFootprintLib:2X5-SHROUDED
- U5: footprint Housings_DIP:DIP-18_W7.62mm -> Housings_DIP:DIP-18_W7.62mm_Socket_LongPads
Connections:
- net VCC: now also B1.VCC, R6.1
- net at U5.1 (SCK): now also SW1.3, SW1.4
- net at U5.2 (SI): now also SW1.5, SW1.6
- net at U5.3 (SO): now also SW1.7, SW1.8
- net at U5.6 (~RESET): now also R6.2
- net at U5.7 (~CS): now also SW1.2
- net at U5.8 (INT): now also SW1.1
- net SCL: now reaches B1.SCL, R1.2
- net SCL: now also SW1.14
- net SDA: now reaches B1.SDA, R2.2
- net SDA: now also SW1.12
- net I2C_A2: now reaches JP1.2, R3.1
- net I2C_A2: now also SW1.10
- net ~CS: now reaches JP4.2
- net ~CS: now also SW1.15
- net SCK: now reaches B1.SCK
- net SCK: now also SW1.13
- net MOSI: now reaches B1.MOSI
- net MOSI: now also SW1.11
- net at B1.D2: now also JP6.3
- net at B1.D3 (*D3): now also JP6.1
- net MISO: now reaches B1.MISO
- net MISO: now also SW1.9
- new net INT: JP6.2, SW1.16
- no-connect marks 26 -> 20
Other:
- moved on the sheet: B1, JP4, JP5
